Commit message: add launch files

File: description/lance.urdf (robot description, URDF)
Before this commit: robot lance, 9 links, 8 joints
Links:
- link collection_link: geometry collision mesh filename=file://$(find csm_gz_sim)/description/lance/meshes/lance-20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; visual mesh filename=file://$(find csm_gz_sim)/description/lance/meshes/lance-20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
- link frame_link: geometry collision mesh filename=file://$(find csm_gz_sim)/description/lance/meshes/lance-20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; visual mesh filename=file://$(find csm_gz_sim)/description/lance/meshes/lance-20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
- link left_track_link: geometry collision mesh filename=file://$(find csm_gz_sim)/description/lance/meshes/lance-20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; visual mesh filename=file://$(find csm_gz_sim)/description/lance/meshes/lance-20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
- link lidar_link: geometry collision cylinder length=0.098 radius=0.048; visual mesh filename=file://$(find csm_gz_sim)/description/lance/meshes/lance-20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
- link right_track_link: geometry collision mesh filename=file://$(find csm_gz_sim)/description/lance/meshes/lance-20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; visual mesh filename=file://$(find csm_gz_sim)/description/lance/meshes/lance-20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

Commit message: discovered the magic numbers

File: description/lance.urdf (robot description, URDF)
Before this commit: robot lance, 9 links, 8 joints
Joints:
- joint lidar_joint: origin xyz=0.64957717 0 0.42478867 rpy=3.1415926 0.3490659 0 -> xyz=0.64957717 0 0.42478867 rpy=2.836255 -0.171851 -2.067879

Commit message: dummy reverse rotated lidar frame

File: description/lance.urdf (robot description, URDF)
Before this commit: robot lance, 9 links, 8 joints
Links:
- added link lidar_link_inv_rotated
Joints:
- added joint lidar_joint_inv_rotated: type fixed, parent lidar_link, child lidar_link_inv_rotated, origin xyz=0 0 0 rpy=0 0 2.09439510239

Commit message: body tags

File: description/lance.urdf (robot description, URDF)
Before this commit: robot lance, 10 links, 9 joints
Links:
- link base_link: geometry visual mesh filename=file://$(find csm_gz_sim)/description/lance/meshes/lance-20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

Commit message: rocks and dump control

File: description/lance.urdf (robot description, URDF)
Before this commit: robot lance, 10 links, 9 joints
Links:
- link frame_link: geometry collision mesh filename=file://$(find csm_gz_sim)/description/lance/meshes/lance-20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; collision mesh filename=file://$(find csm_gz_sim)/description/lance/meshes/lance-20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
